File: sesion2-kovalinskyi/sensores.kicad_sch (KiCad schematic)
At the start: 6 parts, among them U3 MCP9808_MSOP, U4 ADXL343

Commit message: Copia de seguridad Sesión 5
Parts:
- C8, C9: MPN (none) -> CC0805KRX7R9BB104
- R3, R4: MPN (none) -> RC0805FR-074K7L
- U3: MPN (none) -> MCP9808-E/MS
- U4: MPN (none) -> ADXL343BCCZ
Changed lines of the file:
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@@
+			)
+		)
+		(property "MPN" "MCP9808-E/MS"
+			(at 88.9 99.06 0)
+			(hide yes)
+			(show_name no)
+			(do_not_autoplace no)
+			(effects
+				(font
+					(size 1.27 1.27)
+				)
 			)
 		)
@@
 			)
 		)
+		(property "MPN" "CC0805KRX7R9BB104"
+			(at 231.14 71.12 90)
+			(hide yes)
+			(show_name no)
+			(do_not_autoplace no)
+			(effects
+				(font
+					(size 1.27 1.27)
+				)
+			)
+		)
 		(pin "1"
 		)
@@
 			)
 		)
+		(property "MPN" "RC0805FR-074K7L"
+			(at 74.93 85.09 0)
+			(hide yes)
+			(show_name no)
+			(do_not_autoplace no)
+			(effects
+				(font
+					(size 1.27 1.27)
+				)
+			)
+		)
 		(pin "1"
 		)
@@
 			)
 		)
+		(property "MPN" "CC0805KRX7R9BB104"
+			(at 100.33 76.2 90)
+			(hide yes)
+			(show_name no)
+			(do_not_autoplace no)
+			(effects
+				(font
+					(size 1.27 1.27)
+				)
+			)
+		)
 		(pin "1"
 		)
@@
 			)
 		)
+		(property "MPN" "ADXL343BCCZ"
+			(at 220.98 95.25 0)
+			(hide yes)
+			(show_name no)
+			(do_not_autoplace no)
+			(effects
+				(font
+					(size 1.27 1.27)
+				)
+			)
+		)
 		(pin "7"
 		)
@@
 			(at 34.29 87.63 0)
 			(hide yes)
+			(show_name no)
+			(do_not_autoplace no)
+			(effects
+				(font
+					(size 1.27 1.27)
+				)
+			)
+		)
+		(property "MPN" "RC0805FR-074K7L"
+			(at 34.29 87.63 0)
+			(hide yes)
